File: µC Schaltplan/LED_Streifen/streifen.brd (EAGLE design)
At the start: 130 x 30 mm, 22 parts, among them IC1 78L05SMD, IC2 PIC18F2550_28W

Commit message: update to v3
Parts:
- added D2: (no value), diode:DO35-7
- added J1, J2, J3: J5MM, jumper:05
- moved PICKIT3 10.8 mm to (50.2, 12.1)
- moved R3 4.26 mm to (120.7, 18.4)
- moved R2 4.02 mm to (120.7, 14.0)
- moved R1 4.02 mm to (120.7, 10.2)
Connections:
- removed net VSS: BC817.2, BC817_2.2, BC817_3.2, C1.2, C2.2, C3.2, C4.2, IC1.2, IC1.3, IC1.6, IC1.7, IC2.19, IC2.8, JP2.1, PICKIT3.3
- new net GND: BC817_3.2, C1.2, C2.2, C3.2, C4.2, D2.A, IC1.2, IC1.3, IC1.6, IC1.7, IC2.19, IC2.8, IC2.9, J2.2, J3.1, J3.2, JP2.1, PICKIT3.3
- new net N$25: BC817_2.2, J1.2, J2.1
- new net N$26: BC817.2, J1.1
- net N$3: now also D2.C
Routing:
- net VSS: track 81.3 -> 0.00 mm
- net GND: track 0.00 -> 42.7 mm
- net N$7: track 102.5 -> 81.3 mm
- net N$4: track 34.7 -> 23.0 mm
- net N$23: track 19.1 -> 8.07 mm
- net N$24: track 19.7 -> 8.60 mm
- net N$16: track 127.9 -> 119.9 mm
- net N$25: track 0.00 -> 7.81 mm
- net N$26: track 0.00 -> 7.29 mm
- net N$22: track 6.50 -> 10.8 mm
- net N$20: track 6.50 -> 10.6 mm
- net N$21: track 6.50 -> 10.6 mm
- net N$9: track 56.6 -> 58.5 mm
- net N$8: track 66.8 -> 67.5 mm
- added copper zone on layer 1, net GND
- removed copper zone on layer 1, net VSS
Other:
- board text added: "LED Streifen v2 Kat.:20"
- board text removed: "LED Streifen v1 Kat.:20"
