File: µC Schaltplan/LED_Streifen/streifen.sch (EAGLE design)
At the start: 21 parts, among them IC1 78L05SMD, IC2 PIC18F2550_28W

Commit message: update to v3
Parts:
- added D2: (no value), diode:SCHOTTKY-DIODEDO35-7
- added J1, J2, J3: J5MM, jumper:J5MM
Connections:
- removed net VSS: BC817.E, BC817_2.E, BC817_3.E, C1.2, C2.2, C3.2, C4.2, IC1G$1.GND@1, IC1G$1.GND@2, IC1G$1.GND@3, IC1G$1.GND@4, IC2.VSS, IC2.VSS@1, JP2.1, PICKIT3.3
- new net GND: BC817_3.E, C1.2, C2.2, C3.2, C4.2, D2.A, IC1G$1.GND@1, IC1G$1.GND@2, IC1G$1.GND@3, IC1G$1.GND@4, IC2.OSC1/CLKI, IC2.VSS, IC2.VSS@1, J2.2, J3.1, J3.2, JP2.1, PICKIT3.3
- new net N$25: BC817_2.E, J1.2, J2.1
- new net N$26: BC817.E, J1.1
- net N$3: now also D2.C
Changed lines of the file:
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@@
 <part name="R4" library="rcl" deviceset="R-EU_" device="R1206" value="1,2k"/>
 <part name="PICKIT3" library="pinhead" deviceset="PINHD-1X6" device=""/>
+<part name="J1" library="jumper" deviceset="J" device="5MM"/>
+<part name="J2" library="jumper" deviceset="J" device="5MM"/>
+<part name="J3" library="jumper" deviceset="J" device="5MM"/>
+<part name="D2" library="diode" deviceset="SCHOTTKY-DIODE" device="DO35-7"/>
 </parts>
 <sheets>
@@
 <instance part="R4" gate="G$1" x="38.1" y="40.64"/>
 <instance part="PICKIT3" gate="A" x="50.8" y="20.32"/>
+<instance part="J1" gate="1" x="167.64" y="78.74" rot="R270"/>
+<instance part="J2" gate="1" x="167.64" y="63.5" rot="R270"/>
+<instance part="J3" gate="1" x="5.08" y="78.74" rot="R270"/>
+<instance part="D2" gate="G$1" x="10.16" y="63.5" rot="R90"/>
 </instances>
 <busses>
 </busses>
 <nets>
-<net name="VSS" class="0">
-<segment>
-<pinref part="C4" gate="G$1" pin="2"/>
-<wire x1="22.86" y1="91.44" x2="22.86" y2="93.98" width="0.1524" layer="91"/>
-<pinref part="IC1" gate="G$1" pin="GND@4"/>
-<wire x1="10.16" y1="91.44" x2="22.86" y2="91.44" width="0.1524" layer="91"/>
-<pinref part="IC1" gate="G$1" pin="GND@3"/>
-<wire x1="7.62" y1="91.44" x2="10.16" y2="91.44" width="0.1524" layer="91"/>
-<pinref part="IC1" gate="G$1" pin="GND@2"/>
-<wire x1="5.08" y1="91.44" x2="7.62" y2="91.44" width="0.1524" layer="91"/>
-<pinref part="IC1" gate="G$1" pin="GND@1"/>
-<wire x1="2.54" y1="91.44" x2="5.08" y2="91.44" width="0.1524" layer="91"/>
-<pinref part="C1" gate="G$1" pin="2"/>
-<pinref part="C2" gate="G$1" pin="2"/>
-<wire x1="-33.02" y1="96.52" x2="-22.86" y2="96.52" width="0.1524" layer="91"/>
-<pinref part="C3" gate="G$1" pin="2"/>
-<wire x1="-22.86" y1="96.52" x2="-12.7" y2="96.52" width="0.1524" layer="91"/>
-<wire x1="2.54" y1="91.44" x2="-12.7" y2="91.44" width="0.1524" layer="91"/>
-<wire x1="-12.7" y1="91.44" x2="-12.7" y2="96.52" width="0.1524" layer="91"/>
+<net name="GND" class="0">
+<segment>
 <wire x1="-38.1" y1="63.5" x2="5.08" y2="63.5" width="0.1524" layer="91"/>
-<wire x1="5.08" y1="63.5" x2="5.08" y2="91.44" width="0.1524" layer="91"/>
+<wire x1="5.08" y1="63.5" x2="5.08" y2="73.66" width="0.1524" layer="91"/>
 <wire x1="109.22" y1="35.56" x2="30.48" y2="35.56" width="0.1524" layer="91"/>
 <wire x1="30.48" y1="35.56" x2="22.86" y2="35.56" width="0.1524" layer="91"/>
 <wire x1="22.86" y1="35.56" x2="5.08" y2="35.56" width="0.1524" layer="91"/>
-<wire x1="5.08" y1="35.56" x2="5.08" y2="63.5" width="0.1524" layer="91"/>
+<wire x1="5.08" y1="35.56" x2="5.08" y2="60.96" width="0.1524" layer="91"/>
 <junction x="5.08" y="63.5"/>
 <pinref part="IC2" gate="G$1" pin="VSS"/>
+<wire x1="5.08" y1="60.96" x2="5.08" y2="63.5" width="0.1524" layer="91"/>
 <wire x1="104.14" y1="66.04" x2="109.22" y2="66.04" width="0.1524" layer="91"/>
 <wire x1="109.22" y1="66.04" x2="109.22" y2="55.88" width="0.1524" layer="91"/>
@@
 <wire x1="30.48" y1="22.86" x2="30.48" y2="35.56" width="0.1524" layer="91"/>
 <junction x="30.48" y="35.56"/>
-<junction x="-22.86" y="96.52"/>
-<junction x="-12.7" y="96.52"/>
-<junction x="2.54" y="91.44"/>
-<junction x="5.08" y="91.44"/>
-<junction x="7.62" y="91.44"/>
-<junction x="10.16" y="91.44"/>
-<pinref part="BC817_2" gate="G$1" pin="E"/>
-<wire x1="154.94" y1="71.12" x2="167.64" y2="71.12" width="0.1524" layer="91"/>
 <pinref part="BC817_3" gate="G$1" pin="E"/>
 <wire x1="167.64" y1="55.88" x2="154.94" y2="55.88" width="0.1524" layer="91"/>
-<wire x1="167.64" y1="55.88" x2="167.64" y2="71.12" width="0.1524" layer="91"/>
-<junction x="167.64" y="71.12"/>
-<pinref part="BC817" gate="G$1" pin="E"/>
-<wire x1="154.94" y1="86.36" x2="167.64" y2="86.36" width="0.1524" layer="91"/>
-<wire x1="167.64" y1="86.36" x2="167.64" y2="71.12" width="0.1524" layer="91"/>
+<wire x1="167.64" y1="55.88" x2="167.64" y2="58.42" width="0.1524" layer="91"/>
 <wire x1="154.94" y1="55.88" x2="109.22" y2="55.88" width="0.1524" layer="91"/>
 <junction x="109.22" y="55.88"/>
 <junction x="154.94" y="55.88"/>
+<pinref part="IC2" gate="G$1" pin="OSC1/CLKI"/>
+<wire x1="104.14" y1="68.58" x2="109.22" y2="68.58" width="0.1524" layer="91"/>
+<wire x1="109.22" y1="68.58" x2="109.22" y2="66.04" width="0.1524" layer="91"/>
+<junction x="109.22" y="66.04"/>
+<pinref part="J2" gate="1" pin="2"/>
+<pinref part="J3" gate="1" pin="2"/>
+<wire x1="10.16" y1="60.96" x2="5.08" y2="60.96" width="0.1524" layer="91"/>
+<junction x="5.08" y="60.96"/>
+<pinref part="D2" gate="G$1" pin="A"/>
+</segment>
+<segment>
+<pinref part="C3" gate="G$1" pin="2"/>
+<pinref part="C4" gate="G$1" pin="2"/>
+<wire x1="22.86" y1="91.44" x2="22.86" y2="93.98" width="0.1524" layer="91"/>
+<pinref part="IC1" gate="G$1" pin="GND@4"/>
+<wire x1="10.16" y1="91.44" x2="22.86" y2="91.44" width="0.1524" layer="91"/>
+<junction x="10.16" y="91.44"/>
+<pinref part="IC1" gate="G$1" pin="GND@3"/>
+<wire x1="7.62" y1="91.44" x2="10.16" y2="91.44" width="0.1524" layer="91"/>
+<junction x="7.62" y="91.44"/>
+<pinref part="IC1" gate="G$1" pin="GND@2"/>
+<wire x1="5.08" y1="91.44" x2="7.62" y2="91.44" width="0.1524" layer="91"/>
+<pinref part="J3" gate="1" pin="1"/>
+<wire x1="5.08" y1="83.82" x2="5.08" y2="91.44" width="0.1524" layer="91"/>
+<junction x="5.08" y="91.44"/>
+<pinref part="IC1" gate="G$1" pin="GND@1"/>
+<wire x1="2.54" y1="91.44" x2="5.08" y2="91.44" width="0.1524" layer="91"/>
+<junction x="2.54" y="91.44"/>
+<wire x1="2.54" y1="91.44" x2="-12.7" y2="91.44" width="0.1524" layer="91"/>
+<wire x1="-12.7" y1="91.44" x2="-12.7" y2="96.52" width="0.1524" layer="91"/>
+<junction x="-12.7" y="96.52"/>
+<pinref part="C2" gate="G$1" pin="2"/>
+<wire x1="-22.86" y1="96.52" x2="-12.7" y2="96.52" width="0.1524" layer="91"/>
+<junction x="-22.86" y="96.52"/>
+<pinref part="C1" gate="G$1" pin="2"/>
+<wire x1="-33.02" y1="96.52" x2="-22.86" y2="96.52" width="0.1524" layer="91"/>
 </segment>
 </net>
@@
 <segment>
 <pinref part="IC2" gate="G$1" pin="RB0/AN12/INT0/LFT0/SDI/SDA"/>
-<wire x1="27.94" y1="66.04" x2="-38.1" y2="66.04" width="0.1524" layer="91"/>
 <pinref part="JP2" gate="A" pin="2"/>
+<wire x1="27.94" y1="66.04" x2="10.16" y2="66.04" width="0.1524" layer="91"/>
+<pinref part="D2" gate="G$1" pin="C"/>
+<wire x1="10.16" y1="66.04" x2="-38.1" y2="66.04" width="0.1524" layer="91"/>
+<junction x="10.16" y="66.04"/>
 </segment>
 </net>
@@
 </segment>
 </net>
+<net name="N$25" class="0">
+<segment>
+<pinref part="BC817_2" gate="G$1" pin="E"/>
+<wire x1="154.94" y1="71.12" x2="167.64" y2="71.12" width="0.1524" layer="91"/>
+<junction x="167.64" y="71.12"/>
+<pinref part="J2" gate="1" pin="1"/>
+<wire x1="167.64" y1="68.58" x2="167.64" y2="71.12" width="0.1524" layer="91"/>
+<wire x1="167.64" y1="73.66" x2="167.64" y2="71.12" width="0.1524" layer="91"/>
+<pinref part="J1" gate="1" pin="2"/>
+</segment>
+</net>
+<net name="N$26" class="0">
+<segment>
+<pinref part="J1" gate="1" pin="1"/>
+<pinref part="BC817" gate="G$1" pin="E"/>
+<wire x1="154.94" y1="86.36" x2="167.64" y2="86.36" width="0.1524" layer="91"/>
+<wire x1="167.64" y1="86.36" x2="167.64" y2="83.82" width="0.1524" layer="91"/>
+</segment>
+</net>
